File: hardware/kicad/panel/shotpuck-panel.kicad_pcb (KiCad board)
At the start: 2 copper layers, 91 x 92.6 mm, 287 parts, among them J1_0 TYPE-C 6PFS 2JCB1.6-H6.7 IPX8, J1_1 TYPE-C 6PFS 2JCB1.6-H6.7 IPX8, J1_2 TYPE-C 6PFS 2JCB1.6-H6.7 IPX8, J1_3 TYPE-C 6PFS 2JCB1.6-H6.7 IPX8, J2_0 SWD pads, J2_1 SWD pads, J2_2 SWD pads, J2_3 SWD pads, Q1_0 DMN63D8LDW, Q1_1 DMN63D8LDW, Q1_2 DMN63D8LDW, Q1_3 DMN63D8LDW, Q2_0 DMN2004DWK, Q2_1 DMN2004DWK, Q2_2 DMN2004DWK, Q2_3 DMN2004DWK, U1_0 BMD-340-A-R, U1_1 BMD-340-A-R, U1_2 BMD-340-A-R, U1_3 BMD-340-A-R, U2_0 LSM6DSO32TR, U2_1 LSM6DSO32TR, U2_2 LSM6DSO32TR, U2_3 LSM6DSO32TR, U3_0 MCP73831T-2ACI/OT, U3_1 MCP73831T-2ACI/OT, U3_2 MCP73831T-2ACI/OT, U3_3 MCP73831T-2ACI/OT, U4_0 BQ29700DSER, U4_1 BQ29700DSER, U4_2 BQ29700DSER, U4_3 BQ29700DSER

Commit message: Add charger LED, JP2 reset pads and firmware recovery (0.2.1)
Charger LED: one blink every 2 s while charging, steady once the charger
has terminated (so the LED never holds off termination), three blinks
when the temperature gate pauses charging.

JP2: two bare round pads (0.8 mm, 0.4 mm gap) on module pin 7 (P0.26)
and GND. With the cap off, bridging them for 5 s erases settings,
pairings, shot count and log and reboots; only a bridge made while
running counts. Three crash or watchdog resets in a row, each within a
minute of boot, erase the same data automatically. A trial OTA image is
now confirmed only after a paired phone connects over an encrypted link.

Firmware rebuilt and signed as 0.2.1; panel gerbers and JLC BOM/CPL
regenerated (JP2 is copper only).

Co-Authored-By: Claude Opus 5.5 <noreply@anthropic.com>
Parts:
- removed KiKit_MB_12_1, KiKit_MB_16_1, KiKit_MB_4_1, KiKit_MB_8_1: NPTH, NPTH
- added JP2_0: RESET pads, ShotPuck:TweezerPads_2x0.8mm_Gap0.4mm, F.Cu at (117.2, 57.1)
- added JP2_1: RESET pads, ShotPuck:TweezerPads_2x0.8mm_Gap0.4mm, F.Cu at (156.2, 57.1)
- added JP2_2: RESET pads, ShotPuck:TweezerPads_2x0.8mm_Gap0.4mm, F.Cu at (140.8, 75.4)
- added JP2_3: RESET pads, ShotPuck:TweezerPads_2x0.8mm_Gap0.4mm, F.Cu at (179.8, 75.4)
- added KiKit_MB_11_1: NPTH, NPTH, F.Cu at (146.7, 89.8)
- added KiKit_MB_15_1: NPTH, NPTH, F.Cu at (185.7, 89.8)
- added KiKit_MB_3_1: NPTH, NPTH, F.Cu at (111.3, 42.8)
- added KiKit_MB_7_1: NPTH, NPTH, F.Cu at (150.3, 42.8)
- moved KiKit_MB_19_2 75.0 mm to (111.0, 65.8)
- moved KiKit_MB_19_3 75.0 mm to (111.0, 66.8)
- moved KiKit_MB_17_2 37.5 mm to (148.5, 66.8)
- moved KiKit_MB_17_3 37.5 mm to (148.5, 65.8)
- moved KiKit_MB_18_2 37.5 mm to (186.0, 65.8)
- moved KiKit_MB_18_3 37.5 mm to (186.0, 66.8)
- moved KiKit_MB_13_3 34.7 mm to (150.7, 92.1)
- moved KiKit_MB_13_4 34.7 mm to (150.6, 91.4)
- moved KiKit_MB_5_3 34.7 mm to (185.3, 40.4)
- moved KiKit_MB_5_4 34.7 mm to (185.4, 41.2)
- moved KiKit_MB_1_3 34.7 mm to (146.3, 40.4)
- moved KiKit_MB_1_4 34.7 mm to (146.4, 41.2)
- moved KiKit_MB_9_3 34.7 mm to (111.7, 92.1)
- moved KiKit_MB_9_4 34.7 mm to (111.6, 91.4)
- moved KiKit_MB_13_2 34.7 mm to (151.0, 92.9)
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Connections:
- U1_0 pad 7: Board_0-unconnected-(U1-P0.26-Pad7) -> Board_0-/BTN
- U1_1 pad 7: Board_1-unconnected-(U1-P0.26-Pad7) -> Board_1-/BTN
- U1_2 pad 7: Board_2-unconnected-(U1-P0.26-Pad7) -> Board_2-/BTN
- U1_3 pad 7: Board_3-unconnected-(U1-P0.26-Pad7) -> Board_3-/BTN
Routing:
- net Board_0-/GND: track 11.4 -> 26.1 mm, vias 30 -> 31
- net Board_3-/GND: track 11.4 -> 26.1 mm, vias 30 -> 31
- net Board_1-/GND: track 11.4 -> 26.1 mm, vias 30 -> 31
- net Board_2-/GND: track 11.4 -> 26.1 mm, vias 30 -> 31
- net Board_3-/BTN: track 0.00 -> 1.92 mm
- net Board_2-/BTN: track 0.00 -> 1.92 mm
- net Board_0-/BTN: track 0.00 -> 1.92 mm
- net Board_1-/BTN: track 0.00 -> 1.92 mm
- net Board_1-/ACC_INT1: track 5.85 -> 5.28 mm
- net Board_3-/ACC_INT1: track 5.85 -> 5.28 mm
- net Board_2-/ACC_INT1: track 5.85 -> 5.28 mm
- net Board_0-/ACC_INT1: track 5.85 -> 5.28 mm
Other:
- board text added: "RST"
- board text added: "Shotpuck!!1! rev. 0A Richard H. VBK"
