File: hardware/kicad/shotpuck.kicad_pcb (KiCad board)
At the start: 2 copper layers, 36 x 34.8 mm, 36 parts, among them J1 TYPE-C 6PFS 2JCB1.6-H6.7 IPX8, J2 SWD pads, Q1 DMN63D8LDW, Q2 DMN2004DWK, U1 BMD-340-A-R, U2 LSM6DSV32XTR, U3 MCP73831T-2ACI/OT, U4 BQ29700DSER

Commit message: Feed R9 from VIN_RAW and add the hot-plug simulation
A hot-plug simulation of the charge input (324 cases over cable,
supply, C1 derating, D1 and TVS corners) showed that D1 and C1 hold a
plug-in overshoot on VIN for milliseconds, and R9/C9 passes it on to
the nRF VBUS pin: up to 6.36 V against its 5.8 V absolute maximum in
9 cases. Fed from VIN_RAW, before D1, VBUS_SNS stays at or below
5.47 V in every case, and charger detection gains a diode drop of
headroom. R9 sat on VIN only because the magnetic board's hand-wired
lead could be reversed; a USB-C plug cannot reverse VBUS.

- design.py: R9 pin 1 on VIN_RAW.
- shotpuck.kicad_sch: R9 pin-1 label changed in place (gen_sch.py
  would drop the schematic's hand edits). Netlist check PASS, ERC 0
  errors.
- shotpuck.kicad_pcb: R9 pad 1 routed to VIN_RAW by Richard, old VIN
  branch removed. DRC 0/0, 0 schematic-parity issues.
- hardware/hotplug_sim.py: the sweep; --rev-a models the ordered
  boards, which keep R9 on VIN.
- README D27, HANDOVER and VALIDATION updated. The rev A order package
  is unchanged.

Co-Authored-By: Claude Opus 5.5 <noreply@anthropic.com>
Connections:
- R9 pad 1: /VIN -> /VIN_RAW
Routing:
- net /VIN: track 31.6 -> 20.5 mm, vias 7 -> 5
- net /VIN_RAW: track 14.2 -> 15.3 mm
Other:
- board text added: "Båg-pucken rev. 0B Richard H. VBK"
- board text removed: "Båg-pucken rev. 0A Richard H. VBK"
